File: light_curve.kicad_sch (KiCad schematic)
At the start: 151 parts, among them J1 Valve Conn, J10 Valve Conn, J101 Power Input, J102 Servo, J103 Servo, J104 Servo, J105 Servo, J106 Servo, J107 Servo, J108 Servo, J109 Servo, J11 Valve Conn, J110 Servo, J111 Servo, J112 Servo, J113 Servo, J12 Valve Conn, J2 Valve Conn, J21 Power Input, J22 I2C INTERCONNECT, J23 I2C OLED, J24 POLOLU CONVERTER, J25 I2C INTERCONNECT, J26 I2C INTERCONNECT, J27 A2541WV-12P, J28 A2541WV-12P, J3 Valve Conn, J4 Valve Conn, J5 Valve Conn, J6 Valve Conn, J7 Valve Conn, J8 Valve Conn, J9 Valve Conn, Q1 AO3400A, Q10 AO3400A, Q11 AO3400A, Q12 AO3400A, Q2 AO3400A, Q3 AO3400A, Q4 AO3400A, Q5 AO3400A, Q6 AO3400A, Q7 AO3400A, Q8 AO3400A, Q9 AO3400A, SW1 SW_MEC_5G, SW2 SW_MEC_5G, SW22 CONFIG SWITCH, SW3 SW_MEC_5G, U101 USBLC6-2P6, U102 CC6920B, U103 USBLC6-2P6, U104 USBLC6-2P6, U21 TLV1117-50IDCYR, U22 SN74LVC1G07QDCKTQ1, U23 PCA9539PW_118, U24 MOUDLE-SEEEDUINO-XIAO-ESP32S3, U25 PCA9685PW, U26 LSM6DS3, U27 LIS3MDL

Commit message: Update boards for last minute order before the burn! As ordered.
Parts:
- removed C101, C26, C27, C28: 0.1uF, Capacitor_SMD:C_0603_1608Metric, symbol Device:C
- removed C29: 1u, Capacitor_SMD:C_0603_1608Metric, symbol Device:C
- removed JP101, JP103, JP104, JP105, JP21: SolderJumper_2_Open, Jumper:SolderJumper-2_P1.3mm_Open_RoundedPad1.0x1.5mm, symbol Jumper:SolderJumper_2_Open
- removed JP102: Disable Servo Current Measure, symbol Jumper:SolderJumper_2_Bridged
- removed R113: 10k, Resistor_SMD:R_0603_1608Metric, symbol MotorController:TAYLOR_RESISTOR
- removed R54, R55: 5.1k, Resistor_SMD:R_0603_1608Metric, symbol Device:R
- removed U102: CC6920B, Package_SO:SO-8_3.9x4.9mm_P1.27mm, symbol motor_parts:CC6920B
- removed U22: SN74LVC1G07QDCKTQ1, Package_TO_SOT_SMD:SOT-353_SC-70-5, symbol acorn-motherboard:SN74LVC1G07QDCKTQ1
- removed U26: LSM6DS3, Package_LGA:LGA-14_3x2.5mm_P0.5mm_LayoutBorder3x4y, symbol Sensor_Motion:LSM6DS3
- removed U27: LIS3MDL, Package_LGA:LGA-12_2x2mm_P0.5mm, symbol Sensor_Magnetic:LIS3MDL
- added D115, D117, D118: LED_RED, LED_SMD:LED_0603_1608Metric, symbol Device:LED
- added D119, D120: WS2812B, parts:LED_WS2812_3528_3.5x2.8mm_P1.5mm, symbol MotorBuck:WS2812B
- added J114, J115: Conn_01x07, Connector_PinSocket_2.54mm:PinSocket_1x07_P2.54mm_Vertical, symbol Connector_Generic:Conn_01x07
- added Q101: AO7400-VB, Package_TO_SOT_SMD:SOT-323_SC-70, symbol Transistor_FET:AO3400A
- added R114: 130R, Resistor_SMD:R_0603_1608Metric, symbol MotorController:TAYLOR_RESISTOR
- added R115: 402R, Resistor_SMD:R_0603_1608Metric, symbol MotorController:TAYLOR_RESISTOR
- added R116: 1k, Resistor_SMD:R_0603_1608Metric, symbol MotorController:TAYLOR_RESISTOR
- added U102: TXS0101DCKR, Package_TO_SOT_SMD:SOT-363_SC-70-6, symbol MotorBuck:level_shifter
- J22, J25, J26: LCSC C402777 -> C2982033
- J23: value I2C OLED -> OLED
Connections:
- net SERVO_GND is gone; now on net GND: J110.1 (Pin_1), J110.2 (Pin_2), J110.3 (Pin_3), J111.1 (Pin_1), J111.2 (Pin_2), J111.3 (Pin_3), J112.1 (Pin_1), J112.2 (Pin_2), J112.3 (Pin_3), J113.1 (Pin_1), J113.2 (Pin_2), J113.3 (Pin_3)
- net +12V: now also R116.1
- net +3.3V: now also SW22.6, J115.3 (Pin_3), R114.1, U102.1 (VCCA), U102.5 (OE)
- net +5V: now also C102.1, D119.3 (VDD), D120.3 (VDD), U102.6 (VCCB)
- net +6V: now also R115.1
- net A0: no longer SW22.12
- net A1: no longer SW22.11
- net A1_IO: no longer SW22.9
- net A2: now also SW22.9; no longer SW22.10
- net AUX1: now also R44.1, SW1.2, J114.1 (Pin_1)
- net AUX2: now also R46.1, SW2.2, J114.2 (Pin_2)
- net AUX3: now also R49.1, SW3.2, J114.3 (Pin_3)
- net AUX4: now also U23.3 (~RESET), J114.4 (Pin_4)
- net AUX5: now also J114.7 (Pin_7), U102.3 (A)
- net AUX6: now also SW22.12, J115.4 (Pin_4)
- net AUX7: now also SW22.11, J115.5 (Pin_5)
- net AUX8: now also SW22.10, J115.6 (Pin_6)
- net AUX9: now also J115.7 (Pin_7)
- net GND: now also C102.2, R29.2, U25.23 (~{OE}), U25.25 (EXTCLK), J115.2 (Pin_2), Q101.2 (S), U102.2 (GND); no longer C102.1, SW22.6
- net SCL: now also U23.22 (SCL), J114.6 (Pin_6); no longer U23.23 (SDA)
- net SDA: now also U23.23 (SDA), J114.5 (Pin_5); no longer U23.22 (SCL)
- net SW1: no longer R44.1, SW1.2
- net SW2: no longer R46.1, SW2.2
- net SW3: no longer R49.1, SW3.2
- net LED_GND: now reaches D101.1 (K), D102.1 (K), D103.1 (K), D104.1 (K), D105.1 (K), D106.1 (K), D107.1 (K), D108.1 (K), D109.1 (K), D110.1 (K), D111.1 (K), D112.1 (K)
- net LED_GND: now also D115.1 (K), D117.1 (K), D118.1 (K), D119.1 (GND), D120.1 (GND), Q101.3 (D)
- net at D31.1 (K), U24.14 (5V): now also J115.1 (Pin_1)
- net +3V3 renamed LED_EN
- net LED_EN: now also SW22.7, Q101.1 (G)
- removed net /LED_EN: R29.2, SW22.7
- new net: D117.2 (A), R115.2
- new net: D115.2 (A), R114.2
- new net: D119.4 (DOUT), D120.2 (DIN)
- new net: D119.2 (DIN), U102.4 (B)
- new net: D118.2 (A), R116.2
Other:
- note removed: "I2C address"
- note removed: "Motion Sensing"
- moved on the sheet: C23, C24, C25, D1, D10, D101, D102, D103, D104, D105, D106, D107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
